Commit message: Started changes in arm control. Fixed handeye calibrate launch file. Camera_marker frame is not displaying in right place

File: ros_ws/src/iris_ur10e-master/ur_e_description/urdf/aruco.urdf.xacro (robot description, xacro)
@@ -11,5 +11,5 @@
         <origin xyz="0.0 0.0 0.0" rpy="${pi} 0 ${pi/2}"/>
         <geometry>
-          <mesh filename="package://ur_e_description/meshes/aruco/aruco300.dae" scale="1 1 1"/>
+          <mesh filename="package://ur_e_description/meshes/aruco/aruco300.dae" scale="2 2 2"/>
         </geometry>
       </visual>

File: ros_ws/src/iris_ur10e-master/ur_e_description/urdf/ur10e_joint_limited_robot.urdf.xacro (robot description, xacro)
@@ -32,15 +32,14 @@
               rpy="0 0 ${pi/2}"/>
   </xacro:target_chess> -->
-<!--
   <xacro:include filename="$(find ur_e_description)/urdf/aruco.urdf.xacro" />
   <xacro:aruco parent="ee_link" prefix="marker">
       <origin xyz="0.03 0.0 0.04"
               rpy="3.13766148064 0.0 0.0"/>
-  </xacro:aruco> -->
-  <xacro:include filename="$(find ur_e_description)/urdf/charuco.urdf.xacro" />
+  </xacro:aruco>
+  <!-- <xacro:include filename="$(find ur_e_description)/urdf/charuco.urdf.xacro" />
   <xacro:charuco parent="ee_link" prefix="marker">
       <origin xyz="0.15 0.0 0.04"
               rpy="3.13766148064 0.0 0.0"/>
-  </xacro:charuco>
+  </xacro:charuco> -->
   <link name="world" />
   <joint name="world_joint" type="fixed">
