Commit message: Changed xacro file to add camera

File: ros_ws/src/iris_ur10e-master/ur_e_description/urdf/ur10e_joint_limited_robot.urdf.xacro (robot description, xacro)
@@ -16,8 +16,13 @@
 />
   <!-- sensor -->
-  <xacro:include filename="$(find ur_e_description)/urdf/astra.urdf.xacro" />
+  <!-- <xacro:include filename="$(find ur_e_description)/urdf/astra.urdf.xacro" />
   <xacro:sensor_astra parent="ee_link" prefix="camera">
       <origin xyz="0.041311319304504816 -0.06402544453787727 0.044527571211305426"
               rpy="3.13766148064 -0.00787797070144 0.000110993634886"/>
+  </xacro:sensor_astra> -->
+  <xacro:include filename="$(find ur_e_description)/urdf/astra.urdf.xacro" />
+  <xacro:sensor_astra parent="world" prefix="camera">
+      <origin xyz="1 1 1"
+              rpy="0 ${pi/4} -${3*pi/4}"/>
   </xacro:sensor_astra>
   <link name="world" />

Commit message: Added simple target to the simulation.

File: ros_ws/src/iris_ur10e-master/ur_e_description/urdf/ur10e_joint_limited_robot.urdf.xacro (robot description, xacro)
@@ -26,4 +26,10 @@
               rpy="0 ${pi/4} -${3*pi/4}"/>
   </xacro:sensor_astra>
+<!--
+  <xacro:include filename="$(find ur_e_description)/urdf/target.urdf" />
+  <xacro:target_chess parent="gripper_link" prefix="target">
+      <origin xyz="0.15 0 -0.1"
+              rpy="0 0 ${pi/2}"/>
+  </xacro:target_chess> -->
   <link name="world" />
   <joint name="world_joint" type="fixed">

Commit message: aruco model for gazebo

File: ros_ws/src/iris_ur10e-master/ur_e_description/urdf/ur10e_joint_limited_robot.urdf.xacro (robot description, xacro)
@@ -32,4 +32,9 @@
               rpy="0 0 ${pi/2}"/>
   </xacro:target_chess> -->
+  <xacro:include filename="$(find ur_e_description)/urdf/aruco.urdf.xacro" />
+  <xacro:aruco parent="ee_link" prefix="marker">
+      <origin xyz="0.03 0.0 0.04"
+              rpy="3.13766148064 0.0 0.0"/>
+  </xacro:aruco>
   <link name="world" />
   <joint name="world_joint" type="fixed">

Commit message: 7 x 5 charuco model with 30 x 22 cm

File: ros_ws/src/iris_ur10e-master/ur_e_description/urdf/ur10e_joint_limited_robot.urdf.xacro (robot description, xacro)
@@ -23,5 +23,5 @@
   <xacro:include filename="$(find ur_e_description)/urdf/astra.urdf.xacro" />
   <xacro:sensor_astra parent="world" prefix="camera">
-      <origin xyz="1 1 1"
+      <origin xyz="0.75 0.75 0.75"
               rpy="0 ${pi/4} -${3*pi/4}"/>
   </xacro:sensor_astra>
@@ -32,9 +32,15 @@
               rpy="0 0 ${pi/2}"/>
   </xacro:target_chess> -->
+<!--
   <xacro:include filename="$(find ur_e_description)/urdf/aruco.urdf.xacro" />
   <xacro:aruco parent="ee_link" prefix="marker">
       <origin xyz="0.03 0.0 0.04"
               rpy="3.13766148064 0.0 0.0"/>
-  </xacro:aruco>
+  </xacro:aruco> -->
+  <xacro:include filename="$(find ur_e_description)/urdf/charuco.urdf.xacro" />
+  <xacro:charuco parent="ee_link" prefix="marker">
+      <origin xyz="0.15 0.0 0.04"
+              rpy="3.13766148064 0.0 0.0"/>
+  </xacro:charuco>
   <link name="world" />
   <joint name="world_joint" type="fixed">

Commit message: calibration example from visp tutorials

File: ros_ws/src/iris_ur10e-master/ur_e_description/urdf/ur10e_joint_limited_robot.urdf.xacro (robot description, xacro)
@@ -26,20 +26,14 @@
               rpy="0 ${pi/4} -${3*pi/4}"/>
   </xacro:sensor_astra>
-<!--
-  <xacro:include filename="$(find ur_e_description)/urdf/target.urdf" />
-  <xacro:target_chess parent="gripper_link" prefix="target">
-      <origin xyz="0.15 0 -0.1"
-              rpy="0 0 ${pi/2}"/>
-  </xacro:target_chess> -->
-  <xacro:include filename="$(find ur_e_description)/urdf/aruco.urdf.xacro" />
+  <!-- <xacro:include filename="$(find ur_e_description)/urdf/aruco.urdf.xacro" />
   <xacro:aruco parent="ee_link" prefix="marker">
       <origin xyz="0.03 0.0 0.04"
               rpy="3.13766148064 0.0 0.0"/>
-  </xacro:aruco>
-  <!-- <xacro:include filename="$(find ur_e_description)/urdf/charuco.urdf.xacro" />
+  </xacro:aruco> -->
+  <xacro:include filename="$(find ur_e_description)/urdf/charuco.urdf.xacro" />
   <xacro:charuco parent="ee_link" prefix="marker">
       <origin xyz="0.15 0.0 0.04"
               rpy="3.13766148064 0.0 0.0"/>
-  </xacro:charuco> -->
+  </xacro:charuco>
   <link name="world" />
   <joint name="world_joint" type="fixed">
